Commit message: Gazebo Actuator Model Plugin

File: minion_robot/urdf/minion.urdf.xacro (robot description, xacro)
@@ -122,14 +122,50 @@
   <xacro:property name="joint_height" value="0.025"/>
   <!--Left Side-->
-  <xacro:wheel_link id="${lwid}_${ID+1}" radius="${wheel_radius}" thickness="${wheel_thickness}" color="white" mass="${wheel_mass}"/>
+  <xacro:wheel_link id="${lwid}_${ID+1}" radius="${wheel_radius}" thickness="${wheel_thickness}" color="orange" mass="${wheel_mass}"/>
   <xacro:wheel_joint id="blw_${ID+1}" child="${lwid}_${ID+1}" x="${-chassis_length/2+0.03}" y="${chassis_width/2+0.01}" z="${joint_height}"/>
   <xacro:wheel_joint_transmission id="blw_${ID+1}"/>
   <!--Right Side-->
-  <xacro:wheel_link id="${rwid}_${ID+1}" radius="${wheel_radius}" thickness="${wheel_thickness}" color="white" mass="${wheel_mass}"/>
+  <xacro:wheel_link id="${rwid}_${ID+1}" radius="${wheel_radius}" thickness="${wheel_thickness}" color="orange" mass="${wheel_mass}"/>
   <xacro:wheel_joint id="brw_${ID+1}" child="${rwid}_${ID+1}" x="${-chassis_length/2+0.03}" y="${-chassis_width/2-0.01}" z="${joint_height}"/>
   <xacro:wheel_joint_transmission id="brw_${ID+1}"/>
   <gazebo>
-    <plugin name="gazebo_ros_control" filename="libgazebo_ros_control.so">
+<!--     <plugin name="gazebo_ros_control" filename="libgazebo_ros_control.so">
       <robotNamespace>/</robotNamespace>
+    </plugin> -->
+    <plugin name="differential_drive_controller" filename="libgazebo_ros_diff_drive.so">
+     <alwaysOn>true</alwaysOn>
+     <updateRate>20</updateRate>
+     <leftJoint>blw_1</leftJoint>
+     <rightJoint>brw_1</rightJoint>
+     <wheelSeparation>0.2</wheelSeparation>
+     <wheelDiameter>0.07</wheelDiameter>
+     <torque>1.4</torque>
+     <commandTopic>cmd_vel</commandTopic>
+     <odometryTopic>odom</odometryTopic>
+     <odometryFrame>odom</odometryFrame>
+     <robotBaseFrame>base_footprint</robotBaseFrame>
+     <legacyMode>False</legacyMode>
+     </plugin>
+     <plugin name="actuator_plugin_1" filename="libminion_actuator.so">
+      <actuator>
+        <name>actuator_let</name> <!-- optional -->
+        <joint>blw_1</joint> <!-- name of joint to actuate -->
+        <index>0</index> <!-- needed for multi-DOF joints -->
+        <type>electric_motor</type> <!-- motor model type -->
+        <power>5</power> <!-- parameters for motor model -->
+        <max_velocity>15.7</max_velocity>
+        <max_torque>1.4</max_torque>
+      </actuator>
+    </plugin>
+     <plugin name="actuator_plugin_2" filename="libminion_actuator.so">
+      <actuator>
+        <name>actuator_right</name> <!-- optional -->
+        <joint>brw_1</joint> <!-- name of joint to actuate -->
+        <index>0</index> <!-- needed for multi-DOF joints -->
+        <type>electric_motor</type> <!-- motor model type -->
+        <power>5</power> <!-- parameters for motor model -->
+        <max_velocity>15.7</max_velocity>
+        <max_torque>1.4</max_torque>
+      </actuator>
     </plugin>
   </gazebo>

Commit message: Working Battery and Actuator Plugins. pending ROS interface of Actuator with Battery. Namespace issues to be resolved

File: minion_robot/urdf/minion.urdf.xacro (robot description, xacro)
@@ -15,4 +15,8 @@
   <xacro:property name="chassis_width"   value="0.2" />
   <xacro:property name="chassis_height"  value="0.06" />
+  <xacro:property name="battery_mass"    value="0.2" />
+  <xacro:property name="battery_length"  value="0.05" />
+  <xacro:property name="battery_width"   value="0.2" />
+  <xacro:property name="battery_height"  value="0.05" />
   <xacro:property name="wheel_thickness" value="0.02" />
   <xacro:property name="wheel_mass"      value="0.1" />
@@ -90,4 +94,32 @@
     </inertial>
   </link>
+ <!-- <link name="battery_link">
+    <visual>
+      <geometry>
+        <box size="${battery_length} ${battery_width} ${battery_height}"/>
+      </geometry>
+      <origin xyz="0 0 0"/>
+    </visual>
+    <collision>
+      <geometry>
+        <box size="${battery_length} ${battery_width} ${battery_height}"/>
+      </geometry>
+      <origin xyz="0 0 0"/>
+    </collision>
+    <inertial>
+      <mass value="${battery_mass}"/>
+      <inertia ixx="${battery_mass*battery_width*battery_width/12+battery_mass*battery_height*battery_height/12}" ixy="0.0" ixz="0.0"
+        iyy="${battery_mass*battery_length*battery_length/12+battery_mass*battery_height*battery_height/12}" iyz="0.0"
+        izz="${battery_mass*battery_length*battery_length/12+battery_mass*battery_width*battery_width/12}"/>
+    </inertial>
+    <battery name="linear_battery">
+       <voltage>12.592</voltage>
+    </battery>
+ </link>
+ <joint name="battery_base" type="fixed">
+   <parent link="base_link"/>
+   <child link="battery_link"/>
+   <origin xyz="0 0 ${joint_height}"/>
+ </joint>  -->
   <link name="castor">
     <visual>
@@ -169,4 +201,21 @@
       </actuator>
     </plugin>
+<!--     <plugin name="battery" filename="libminion_battery.so">
+        <ros_node>battery_monitor_client</ros_node>
+        <link_name>battery_link</link_name>
+        <battery_name>linear_battery</battery_name>
+        <constant_coef>12.694</constant_coef>
+        <linear_coef>-100.1424</linear_coef>
+        <initial_charge>1.1665</initial_charge>
+        <capacity>1.2009</capacity>
+        <resistance>0.061523</resistance>
+        <smooth_current_tau>1.9499</smooth_current_tau>
+        <charge_rate>0.2</charge_rate>
+    </plugin>
+    <plugin name="consumer" filename="libminion_battery_consumer.so">
+        <link_name>battery_link</link_name>
+        <battery_name>linear_battery</battery_name>
+        <power_load>6.6</power_load>
+    </plugin>     -->
   </gazebo>
 </robot>

Commit message: modified urdf

File: minion_robot/urdf/minion.urdf.xacro (robot description, xacro)
@@ -11,4 +11,5 @@
   </material>
   <!-- Constants-->
+  <xacro:property name="namespace"       value="$(arg namespace)" />
   <xacro:property name="chassis_mass"    value="2" />
   <xacro:property name="chassis_length"  value="0.25" />
@@ -21,4 +22,10 @@
   <xacro:property name="wheel_thickness" value="0.02" />
   <xacro:property name="wheel_mass"      value="0.1" />
+  <!-- More Constants -->
+  <xacro:property name="lwid" value="left_wheel"/>
+  <xacro:property name="rwid" value="right_wheel"/>
+  <xacro:property name="ID" value="0"/>
+  <xacro:property name="wheel_radius" value="0.035"/>
+  <xacro:property name="joint_height" value="0.025"/>
   <xacro:macro name="wheel_inertia" params="mass">
       <inertial>
@@ -54,5 +61,5 @@
   <xacro:macro name="wheel_joint" params="id child x y z">
    <joint name="${id}" type="continuous">
-     <parent link="base_link"/>
+     <parent link="${namespace}/base_link"/>
      <child link="${child}"/>
      <origin xyz="${x} ${y} ${z}"/>
@@ -73,5 +80,5 @@
   </transmission>
   </xacro:macro>
-  <link name="base_link">
+  <link name="${namespace}/base_link">
     <visual>
       <geometry>
@@ -94,33 +101,5 @@
     </inertial>
   </link>
- <!-- <link name="battery_link">
-    <visual>
-      <geometry>
-        <box size="${battery_length} ${battery_width} ${battery_height}"/>
-      </geometry>
-      <origin xyz="0 0 0"/>
-    </visual>
-    <collision>
-      <geometry>
-        <box size="${battery_length} ${battery_width} ${battery_height}"/>
-      </geometry>
-      <origin xyz="0 0 0"/>
-    </collision>
-    <inertial>
-      <mass value="${battery_mass}"/>
-      <inertia ixx="${battery_mass*battery_width*battery_width/12+battery_mass*battery_height*battery_height/12}" ixy="0.0" ixz="0.0"
-        iyy="${battery_mass*battery_length*battery_length/12+battery_mass*battery_height*battery_height/12}" iyz="0.0"
-        izz="${battery_mass*battery_length*battery_length/12+battery_mass*battery_width*battery_width/12}"/>
-    </inertial>
-    <battery name="linear_battery">
-       <voltage>12.592</voltage>
-    </battery>
- </link>
- <joint name="battery_base" type="fixed">
-   <parent link="base_link"/>
-   <child link="battery_link"/>
-   <origin xyz="0 0 ${joint_height}"/>
- </joint>  -->
-  <link name="castor">
+   <link name="${namespace}/castor">
     <visual>
       <geometry>
@@ -142,30 +121,24 @@
     </gazebo>
   </link>
-  <joint name="base_castor" type="fixed">
-     <parent link="base_link"/>
-     <child link="castor"/>
+  <joint name="${namespace}/base_castor" type="fixed">
+     <parent link="${namespace}/base_link"/>
+     <child link="${namespace}/castor"/>
      <origin xyz="${chassis_length/2-wheel_radius} 0 ${joint_height}"/>
   </joint>
-  <!-- More Constants -->
-  <xacro:property name="lwid" value="left_wheel"/>
-  <xacro:property name="rwid" value="right_wheel"/>
-  <xacro:property name="ID" value="0"/>
-  <xacro:property name="wheel_radius" value="0.035"/>
-  <xacro:property name="joint_height" value="0.025"/>
   <!--Left Side-->
-  <xacro:wheel_link id="${lwid}_${ID+1}" radius="${wheel_radius}" thickness="${wheel_thickness}" color="orange" mass="${wheel_mass}"/>
-  <xacro:wheel_joint id="blw_${ID+1}" child="${lwid}_${ID+1}" x="${-chassis_length/2+0.03}" y="${chassis_width/2+0.01}" z="${joint_height}"/>
-  <xacro:wheel_joint_transmission id="blw_${ID+1}"/>
+  <xacro:wheel_link id="${namespace}/${lwid}_${ID+1}" radius="${wheel_radius}" thickness="${wheel_thickness}" color="orange" mass="${wheel_mass}"/>
+  <xacro:wheel_joint id="${namespace}/blw_${ID+1}" child="${namespace}/${lwid}_${ID+1}" x="${-chassis_length/2+0.03}" y="${chassis_width/2+0.01}" z="${joint_height}"/>
+  <xacro:wheel_joint_transmission id="${namespace}/blw_${ID+1}"/>
   <!--Right Side-->
-  <xacro:wheel_link id="${rwid}_${ID+1}" radius="${wheel_radius}" thickness="${wheel_thickness}" color="orange" mass="${wheel_mass}"/>
-  <xacro:wheel_joint id="brw_${ID+1}" child="${rwid}_${ID+1}" x="${-chassis_length/2+0.03}" y="${-chassis_width/2-0.01}" z="${joint_height}"/>
-  <xacro:wheel_joint_transmission id="brw_${ID+1}"/>
+  <xacro:wheel_link id="${namespace}/${rwid}_${ID+1}" radius="${wheel_radius}" thickness="${wheel_thickness}" color="orange" mass="${wheel_mass}"/>
+  <xacro:wheel_joint id="${namespace}/brw_${ID+1}" child="${namespace}/${rwid}_${ID+1}" x="${-chassis_length/2+0.03}" y="${-chassis_width/2-0.01}" z="${joint_height}"/>
+  <xacro:wheel_joint_transmission id="${namespace}/brw_${ID+1}"/>
   <gazebo>
-<!--     <plugin name="gazebo_ros_control" filename="libgazebo_ros_control.so">
+    <plugin name="gazebo_ros_control" filename="libgazebo_ros_control.so">
       <robotNamespace>/</robotNamespace>
-    </plugin> -->
-    <plugin name="differential_drive_controller" filename="libgazebo_ros_diff_drive.so">
+    </plugin>
+    <!-- <plugin name="differential_drive_controller" filename="libgazebo_ros_diff_drive.so">
      <alwaysOn>true</alwaysOn>
-     <updateRate>20</updateRate>
+     <updateRate>10</updateRate>
      <leftJoint>blw_1</leftJoint>
      <rightJoint>brw_1</rightJoint>
@@ -178,27 +151,27 @@
      <robotBaseFrame>base_footprint</robotBaseFrame>
      <legacyMode>False</legacyMode>
-     </plugin>
-     <plugin name="actuator_plugin_1" filename="libminion_actuator.so">
+     </plugin> -->
+<!--      <plugin name="actuator_plugin_1" filename="libminion_actuator.so">
       <actuator>
-        <name>actuator_let</name> <!-- optional -->
-        <joint>blw_1</joint> <!-- name of joint to actuate -->
-        <index>0</index> <!-- needed for multi-DOF joints -->
-        <type>electric_motor</type> <!-- motor model type -->
-        <power>5</power> <!-- parameters for motor model -->
+        <name>actuator_left</name>
+        <joint>blw_1</joint>
+        <index>0</index>
+        <type>electric_motor</type>
+        <power>5</power>
         <max_velocity>15.7</max_velocity>
         <max_torque>1.4</max_torque>
       </actuator>
-    </plugin>
-     <plugin name="actuator_plugin_2" filename="libminion_actuator.so">
+    </plugin> -->
+<!--      <plugin name="actuator_plugin_2" filename="libminion_actuator.so">
       <actuator>
-        <name>actuator_right</name> <!-- optional -->
-        <joint>brw_1</joint> <!-- name of joint to actuate -->
-        <index>0</index> <!-- needed for multi-DOF joints -->
-        <type>electric_motor</type> <!-- motor model type -->
-        <power>5</power> <!-- parameters for motor model -->
+        <name>actuator_right</name>
+        <joint>brw_1</joint>
+        <index>0</index>
+        <type>electric_motor</type>
+        <power>5</power>
         <max_velocity>15.7</max_velocity>
         <max_torque>1.4</max_torque>
       </actuator>
-    </plugin>
+    </plugin>     -->
 <!--     <plugin name="battery" filename="libminion_battery.so">
         <ros_node>battery_monitor_client</ros_node>

Commit message: Lab PC trials

File: minion_robot/urdf/minion.urdf.xacro (robot description, xacro)
@@ -61,5 +61,5 @@
   <xacro:macro name="wheel_joint" params="id child x y z">
    <joint name="${id}" type="continuous">
-     <parent link="${namespace}/base_link"/>
+     <parent link="base_link"/>
      <child link="${child}"/>
      <origin xyz="${x} ${y} ${z}"/>
@@ -80,5 +80,5 @@
   </transmission>
   </xacro:macro>
-  <link name="${namespace}/base_link">
+  <link name="base_link">
     <visual>
       <geometry>
@@ -101,5 +101,5 @@
     </inertial>
   </link>
-   <link name="${namespace}/castor">
+   <link name="castor">
     <visual>
       <geometry>
@@ -121,74 +121,74 @@
     </gazebo>
   </link>
-  <joint name="${namespace}/base_castor" type="fixed">
-     <parent link="${namespace}/base_link"/>
-     <child link="${namespace}/castor"/>
+  <joint name="base_castor" type="fixed">
+     <parent link="base_link"/>
+     <child link="castor"/>
      <origin xyz="${chassis_length/2-wheel_radius} 0 ${joint_height}"/>
   </joint>
   <!--Left Side-->
-  <xacro:wheel_link id="${namespace}/${lwid}_${ID+1}" radius="${wheel_radius}" thickness="${wheel_thickness}" color="orange" mass="${wheel_mass}"/>
-  <xacro:wheel_joint id="${namespace}/blw_${ID+1}" child="${namespace}/${lwid}_${ID+1}" x="${-chassis_length/2+0.03}" y="${chassis_width/2+0.01}" z="${joint_height}"/>
-  <xacro:wheel_joint_transmission id="${namespace}/blw_${ID+1}"/>
+  <xacro:wheel_link id="${lwid}_${ID+1}" radius="${wheel_radius}" thickness="${wheel_thickness}" color="orange" mass="${wheel_mass}"/>
+  <xacro:wheel_joint id="blw_${ID+1}" child="${lwid}_${ID+1}" x="${-chassis_length/2+0.03}" y="${chassis_width/2+0.01}" z="${joint_height}"/>
+  <xacro:wheel_joint_transmission id="blw_${ID+1}"/>
   <!--Right Side-->
-  <xacro:wheel_link id="${namespace}/${rwid}_${ID+1}" radius="${wheel_radius}" thickness="${wheel_thickness}" color="orange" mass="${wheel_mass}"/>
-  <xacro:wheel_joint id="${namespace}/brw_${ID+1}" child="${namespace}/${rwid}_${ID+1}" x="${-chassis_length/2+0.03}" y="${-chassis_width/2-0.01}" z="${joint_height}"/>
-  <xacro:wheel_joint_transmission id="${namespace}/brw_${ID+1}"/>
+  <xacro:wheel_link id="${rwid}_${ID+1}" radius="${wheel_radius}" thickness="${wheel_thickness}" color="orange" mass="${wheel_mass}"/>
+  <xacro:wheel_joint id="brw_${ID+1}" child="${rwid}_${ID+1}" x="${-chassis_length/2+0.03}" y="${-chassis_width/2-0.01}" z="${joint_height}"/>
+  <xacro:wheel_joint_transmission id="brw_${ID+1}"/>
   <gazebo>
     <plugin name="gazebo_ros_control" filename="libgazebo_ros_control.so">
-      <robotNamespace>/</robotNamespace>
+      <robotNamespace>/${namespace}/diff_drive_controller</robotNamespace>
     </plugin>
-    <!-- <plugin name="differential_drive_controller" filename="libgazebo_ros_diff_drive.so">
-     <alwaysOn>true</alwaysOn>
-     <updateRate>10</updateRate>
-     <leftJoint>blw_1</leftJoint>
-     <rightJoint>brw_1</rightJoint>
-     <wheelSeparation>0.2</wheelSeparation>
-     <wheelDiameter>0.07</wheelDiameter>
-     <torque>1.4</torque>
-     <commandTopic>cmd_vel</commandTopic>
-     <odometryTopic>odom</odometryTopic>
-     <odometryFrame>odom</odometryFrame>
-     <robotBaseFrame>base_footprint</robotBaseFrame>
-     <legacyMode>False</legacyMode>
-     </plugin> -->
-<!--      <plugin name="actuator_plugin_1" filename="libminion_actuator.so">
-      <actuator>
-        <name>actuator_left</name>
-        <joint>blw_1</joint>
-        <index>0</index>
-        <type>electric_motor</type>
-        <power>5</power>
-        <max_velocity>15.7</max_velocity>
-        <max_torque>1.4</max_torque>
-      </actuator>
-    </plugin> -->
-<!--      <plugin name="actuator_plugin_2" filename="libminion_actuator.so">
-      <actuator>
-        <name>actuator_right</name>
-        <joint>brw_1</joint>
-        <index>0</index>
-        <type>electric_motor</type>
-        <power>5</power>
-        <max_velocity>15.7</max_velocity>
-        <max_torque>1.4</max_torque>
-      </actuator>
-    </plugin>     -->
-<!--     <plugin name="battery" filename="libminion_battery.so">
-        <ros_node>battery_monitor_client</ros_node>
-        <link_name>battery_link</link_name>
-        <battery_name>linear_battery</battery_name>
-        <constant_coef>12.694</constant_coef>
-        <linear_coef>-100.1424</linear_coef>
-        <initial_charge>1.1665</initial_charge>
-        <capacity>1.2009</capacity>
-        <resistance>0.061523</resistance>
-        <smooth_current_tau>1.9499</smooth_current_tau>
-        <charge_rate>0.2</charge_rate>
-    </plugin>
-    <plugin name="consumer" filename="libminion_battery_consumer.so">
-        <link_name>battery_link</link_name>
-        <battery_name>linear_battery</battery_name>
-        <power_load>6.6</power_load>
-    </plugin>     -->
   </gazebo>
 </robot>
+<!-- <plugin name="differential_drive_controller" filename="libgazebo_ros_diff_drive.so">
+ <alwaysOn>true</alwaysOn>
+ <updateRate>10</updateRate>
+ <leftJoint>blw_1</leftJoint>
+ <rightJoint>brw_1</rightJoint>
+ <wheelSeparation>0.2</wheelSeparation>
+ <wheelDiameter>0.07</wheelDiameter>
+ <torque>1.4</torque>
+ <commandTopic>cmd_vel</commandTopic>
+ <odometryTopic>odom</odometryTopic>
+ <odometryFrame>odom</odometryFrame>
+ <robotBaseFrame>base_footprint</robotBaseFrame>
+ <legacyMode>False</legacyMode>
+ </plugin> -->
+<!--      <plugin name="actuator_plugin_1" filename="libminion_actuator.so">
+  <actuator>
+    <name>actuator_left</name>
+    <joint>blw_1</joint>
+    <index>0</index>
+    <type>electric_motor</type>
+    <power>5</power>
+    <max_velocity>15.7</max_velocity>
+    <max_torque>1.4</max_torque>
+  </actuator>
+</plugin> -->
+<!--      <plugin name="actuator_plugin_2" filename="libminion_actuator.so">
+  <actuator>
+    <name>actuator_right</name>
+    <joint>brw_1</joint>
+    <index>0</index>
+    <type>electric_motor</type>
+    <power>5</power>
+    <max_velocity>15.7</max_velocity>
+    <max_torque>1.4</max_torque>
+  </actuator>
+</plugin>     -->
+<!--     <plugin name="battery" filename="libminion_battery.so">
+    <ros_node>battery_monitor_client</ros_node>
+    <link_name>battery_link</link_name>
+    <battery_name>linear_battery</battery_name>
+    <constant_coef>12.694</constant_coef>
+    <linear_coef>-100.1424</linear_coef>
+    <initial_charge>1.1665</initial_charge>
+    <capacity>1.2009</capacity>
+    <resistance>0.061523</resistance>
+    <smooth_current_tau>1.9499</smooth_current_tau>
+    <charge_rate>0.2</charge_rate>
+</plugin>
+<plugin name="consumer" filename="libminion_battery_consumer.so">
+    <link_name>battery_link</link_name>
+    <battery_name>linear_battery</battery_name>
+    <power_load>6.6</power_load>
+</plugin>     -->

Commit message: Gazebo-Ros-Minion Battery and Formation

File: minion_robot/urdf/minion.urdf.xacro (robot description, xacro)
@@ -56,5 +56,5 @@
       <kp value="10000000.0" />
       <kd value="1.0" />
-      <material>Gazebo/Grey</material>
+      <material>Gazebo/White</material>
     </gazebo>
   </xacro:macro>
@@ -101,4 +101,7 @@
     </inertial>
   </link>
+  <gazebo reference="base_link">
+    <material>Gazebo/Orange</material>
+  </gazebo>
    <link name="castor">
     <visual>
@@ -113,12 +116,12 @@
       </geometry>
     </collision>
-    <gazebo reference="castor">
-      <slip1 value="1"/>
-      <slip2 value="1"/>
-      <kp value="10000000.0" />
-      <kd value="1.0" />
-      <material>Gazebo/Grey</material>
-    </gazebo>
   </link>
+  <gazebo reference="castor">
+    <slip1 value="1"/>
+    <slip2 value="1"/>
+    <kp value="10000000.0" />
+    <kd value="1.0" />
+    <material>Gazebo/Grey</material>
+  </gazebo>
   <joint name="base_castor" type="fixed">
      <parent link="base_link"/>
@@ -136,5 +139,4 @@
   <gazebo>
     <plugin name="gazebo_ros_control" filename="libgazebo_ros_control.so">
-      <robotNamespace>/${namespace}/diff_drive_controller</robotNamespace>
     </plugin>
   </gazebo>
